File: KiCad/MZ-2000_SD/MZ2000_SD.kicad_pcb (KiCad board)
At the start: 2 copper layers, 100 x 100 mm, 21 parts, among them J1 BUS, J2 Micro_SD_Card_Kit, U1 74LS273, U2 74LS273, U3 8255, U4 Arduino_Pro_Mini_5V, U5 GAL22V10, U6 29C256/27C512, U9 74LS245

Commit message: Add files via upload
Connections:
- net Net-(J1-Pada14) renamed /A7
- net Net-(J1-Pada15) renamed /A6
- net Net-(J1-Pada16) renamed /A5
- net Net-(J1-Pada17) renamed /A4
- net Net-(J1-Pada18) renamed /A3
- net Net-(J1-Pada19) renamed /A2
- net Net-(J1-Pada2) renamed /D2
- net Net-(J1-Pada20) renamed /A1
- net Net-(J1-Pada21) renamed /A0
- net Net-(J1-Pada3) renamed /D1
- net Net-(J1-Pada4) renamed /D0
- net Net-(J1-Padb10) renamed /~RD
- net Net-(J1-Padb11) renamed /~IOREQ
- net Net-(J1-Padb17) renamed /RESET
- net Net-(J1-Padb2) renamed /D3
- net Net-(J1-Padb3) renamed /D4
- net Net-(J1-Padb4) renamed /D5
- net Net-(J1-Padb5) renamed /D6
- net Net-(J1-Padb6) renamed /D7
- net Net-(J1-Padb9) renamed /~WR

Commit message: Add files via upload
Parts:
- added J3: MicroSD Card Adapter, Connector_PinSocket_2.54mm:PinSocket_1x06_P2.54mm_Vertical, F.Cu at (149.2, 83.8)
Connections:
- net Net-(J2-Pad5) renamed /SCK
- net Net-(J2-Pad6) renamed /MISO
- net Net-(J2-Pad7) renamed /MOSI
- net Net-(J2-Pad8) renamed /CS
Routing:
- net /SCK: track 38.1 -> 54.8 mm
- net /MOSI: track 32.2 -> 42.1 mm
- net /MISO: track 34.5 -> 44.3 mm
- net /CS: track 29.8 -> 38.6 mm
- net GND: track 394.5 -> 398.5 mm
- net +5V: track 304.9 -> 307.2 mm
- net Net-(S1-Pad2): track 67.3 -> 68.2 mm
Other:
- board text added: "+5V"
- board text added: "CS"
- board text added: "MISO"
- board text added: "MOSI"
- board text added: "MZ-2000 SD-CARD UNIT Rev2.3"
- board text added: "MicroSD Card Adapter"
- board text added: "SCK"
- board text removed: "MZ-2000 SD-CARD UNIT Rev2.2"
