File: KiCad/MZ-2000_SD/MZ2000_SD.sch (KiCad schematic (older format))
At the start: 17 parts, among them J1 BUS, J2 Micro_SD_Card_Kit, U1 74LS273, U2 74LS273, U3 8255, U4 Arduino_Pro_Mini_5V, U5 GAL22V10, U6 29C256/27C512, U9 74LS245

Commit message: Add files via upload
Connections:
- net D7: now reaches J1.b6 (Pin_b6), U1.18 (D7), U2.18 (D7), U3.27 (D7), U9.9 (A7)
- net D6: now reaches J1.b5 (Pin_b5), U1.17 (D6), U2.17 (D6), U3.28 (D6), U9.8 (A6)
- net D5: now reaches J1.b4 (Pin_b4), U1.14 (D5), U2.14 (D5), U3.29 (D5), U9.7 (A5)
- net D4: now reaches J1.b3 (Pin_b3), U1.13 (D4), U2.13 (D4), U3.30 (D4), U9.6 (A4)
- net D3: now reaches J1.b2 (Pin_b2), U1.8 (D3), U2.8 (D3), U3.31 (D3), U9.5 (A3)
- net D2: now reaches J1.a2 (Pin_a2), U1.7 (D2), U2.7 (D2), U3.32 (D2), U9.4 (A2)
- net D1: now reaches J1.a3 (Pin_a3), U1.4 (D1), U2.4 (D1), U3.33 (D1), U9.3 (A1)
- net D0: now reaches J1.a4 (Pin_a4), U1.3 (D0), U2.3 (D0), U3.34 (D0), U9.2 (A0)
- net RESET: now reaches J1.b17 (Pin_b17), U3.35 (RESET), U5.14 (IO10)
- net ~WR: now reaches J1.b9 (Pin_b9), U3.36 (~WR~), U5.10 (I10)
- net ~RD: now reaches J1.b10 (Pin_b10), U3.5 (~RD~), U5.9 (I9)
- net A1: now reaches J1.a20 (Pin_a20), U3.8 (A1), U5.2 (I2)
- net A0: now reaches J1.a21 (Pin_a21), U3.9 (A0), U5.1 (I1/CLK)
- net A7: now reaches J1.a14 (Pin_a14), U5.8 (I8)
- net A6: now reaches J1.a15 (Pin_a15), U5.7 (I7)
- net A5: now reaches J1.a16 (Pin_a16), U5.6 (I6)
- net A4: now reaches J1.a17 (Pin_a17), U5.5 (I5)
- net A3: now reaches J1.a18 (Pin_a18), U5.4 (I4/PD)
- net A2: now reaches J1.a19 (Pin_a19), U5.3 (I3)
- net ~IOREQ: now reaches J1.b11 (Pin_b11), U5.11 (I11)
Other:
- moved on the sheet: C1

Commit message: Add files via upload
Parts:
- added J3: MicroSD Card Adapter, Connector_PinSocket_2.54mm:PinSocket_1x06_P2.54mm_Vertical, symbol Connector_Generic:Conn_01x06
Connections:
- net +5V: now also J3.2 (Pin_2)
- net GND: now also J3.1 (Pin_1)
- net CS: now reaches J2.8 (CS), U4.13 (~~D10)
- net CS: now also J3.6 (Pin_6)
- net MOSI: now reaches J2.7 (CMD), U4.14 (~~D11)
- net MOSI: now also J3.4 (Pin_4)
- net MISO: now reaches J2.6 (DAT), U4.15 (D12)
- net MISO: now also J3.3 (Pin_3)
- net SCK: now reaches J2.5 (CLK), U4.16 (D13)
- net SCK: now also J3.5 (Pin_5)
Changed lines of the file:
@@
 Title "MZ-2000_SD"
 Date ""
-Rev "Rev2.2"
+Rev "Rev2.3"
 Comp ""
 Comment1 ""
@@
 Wire Wire Line
 	2650 9200 2900 9200
+Text Label 12950 3450 0    50   ~ 0
+SCK
+Text Label 12950 3550 0    50   ~ 0
+MISO
+Text Label 12950 3650 0    50   ~ 0
+MOSI
+Text Label 12950 3750 0    50   ~ 0
+CS
+$Comp
+L Connector_Generic:Conn_01x06 J3
+U 1 1 62C204C0
+P 14050 4600
+F 0 "J3" H 14130 4592 50  0000 L CNN
+F 1 "MicroSD Card Adapter" H 13650 4100 50  0000 L CNN
+F 2 "Connector_PinSocket_2.54mm:PinSocket_1x06_P2.54mm_Vertical" H 14050 4600 50  0001 C CNN
+F 3 "~" H 14050 4600 50  0001 C CNN
+	1    14050 4600
+	1    0    0    -1
+$EndComp
+Wire Wire Line
+	13850 4400 13650 4400
+Wire Wire Line
+	13850 4500 13650 4500
+Wire Wire Line
+	13850 4600 13650 4600
+Wire Wire Line
+	13850 4700 13650 4700
+Wire Wire Line
+	13850 4800 13650 4800
+Wire Wire Line
+	13850 4900 13650 4900
+Text Label 13650 4400 0    50   ~ 0
+GND
+Text Label 13650 4500 0    50   ~ 0
++5V
+Text Label 13650 4600 0    50   ~ 0
+MISO
+Text Label 13650 4700 0    50   ~ 0
+MOSI
+Text Label 13650 4800 0    50   ~ 0
+SCK
+Text Label 13650 4900 0    50   ~ 0
+CS
 $EndSCHEMATC
