File: KiCad/MZ-2000_EXT-BOARD/mz-2000.kicad_pcb (KiCad board)
At the start: 2 copper layers, 100 x 99.8 mm, 5 parts, among them J1 Conn_02x22_Row_Letter_First, J2 Conn_02x22_Row_Letter_First, J4 Jack-DC, J5 Conn_02x22_Row_Letter_First

Commit message: Add files via upload
Parts:
- added MH1: MountingHole_3.2mm_M3, MountingHole:MountingHole_3.2mm_M3, F.Cu at (55.0, 150.0)
- added MH2: MountingHole_3.2mm_M3, MountingHole:MountingHole_3.2mm_M3, F.Cu at (145.0, 150.0)
- added MH3: MountingHole_3.2mm_M3, MountingHole:MountingHole_3.2mm_M3, F.Cu at (55.0, 76.0)

Commit message: Add files via upload
Parts:
- removed MH1, MH2, MH3: MountingHole_3.2mm_M3, MountingHole:MountingHole_3.2mm_M3
- S1: value ON OFF -> OFF ON
Connections:
- net Net-(J1-Pada10) renamed /A11
- net Net-(J1-Pada11) renamed /A10
- net Net-(J1-Pada12) renamed /A9
- net Net-(J1-Pada13) renamed /A8
- net Net-(J1-Pada14) renamed /A7
- net Net-(J1-Pada15) renamed /A6
- net Net-(J1-Pada16) renamed /A5
- net Net-(J1-Pada17) renamed /A4
- net Net-(J1-Pada18) renamed /A3
- net Net-(J1-Pada19) renamed /A2
- net Net-(J1-Pada2) renamed /D2
- net Net-(J1-Pada20) renamed /A1
- net Net-(J1-Pada21) renamed /A0
- net Net-(J1-Pada3) renamed /D1
- net Net-(J1-Pada4) renamed /D0
- net Net-(J1-Pada6) renamed /A15
- net Net-(J1-Pada7) renamed /A14
- net Net-(J1-Pada8) renamed /A13
- net Net-(J1-Pada9) renamed /A12
- net Net-(J1-Padb10) renamed /~RD
- net Net-(J1-Padb11) renamed /~IOREQ
- net Net-(J1-Padb12) renamed /~MREQ
- net Net-(J1-Padb14) renamed /~HALT
- net Net-(J1-Padb15) renamed /IE1
- net Net-(J1-Padb16) renamed /IE0
- net Net-(J1-Padb17) renamed /RESET
- net Net-(J1-Padb18) renamed /~EXRESET
- net Net-(J1-Padb19) renamed /~EXINT
- net Net-(J1-Padb2) renamed /D3
- net Net-(J1-Padb20) renamed /~EXWAIT
- net Net-(J1-Padb21) renamed /~MNI
- net Net-(J1-Padb3) renamed /D4
- net Net-(J1-Padb4) renamed /D5
- net Net-(J1-Padb5) renamed /D6
- net Net-(J1-Padb6) renamed /D7
- net Net-(J1-Padb7) renamed /Φ
- net Net-(J1-Padb8) renamed /~M1
- net Net-(J1-Padb9) renamed /~WR

Commit message: Add files via upload
Connections:
- net /Φ renamed /phi
Other:
- board text added: "ON OFF"
- board text added: "phi"
- board text removed: "Φ"
