File: KiCad/MZ-80B_EXT-BOARD/mz-80b.kicad_pcb (KiCad board)
At the start: 2 copper layers, 100 x 99.8 mm, 10 parts, among them J1 Conn_02x22_Row_Letter_First, J2 Conn_02x22_Row_Letter_First, J3 Conn_01x01, J4 Jack-DC, J5 Conn_02x20_Odd_Even

Commit message: Add files via upload
Parts:
- removed MH2, MH3, MH4: MountingHole_3.2mm_M3, MountingHole:MountingHole_3.2mm_M3
